Commit message: fix: enforce canonical spherehand training pipeline

File: src/holosoma/holosoma/data/robots/g1/g1_29dof_spherehand.urdf (robot description, URDF)
Before this commit: robot g1_29dof, 53 links, 52 joints
Links:
- link right_ankle_roll_link: geometry collision mesh filename=assets/right_ankle_roll_link.obj; visual mesh filename=assets/right_ankle_roll_link.obj
